Commit message: Successful grasp

File: hand_full_control/robot/soft_hand_full_actuation.urdf.xacro (robot description, xacro)
@@ -2,4 +2,5 @@
 <robot xmlns:xacro="http://www.ros.org/wiki/xacro" name="soft_hand">
 	<xacro:include filename="$(find soft_hand_description)/model/soft_hand.urdf.xacro"/>
+	<link name="world"/>
 	<link name="box">
 		<inertial>
@@ -24,4 +25,5 @@
 		<material>Gazebo/Wood</material>
 	</gazebo>
+	<joint name="world_to_box" type="fixed"> <parent link="world"/> <child link="box"/> <origin xyz="0 0 0" rpy="0 0 0" /> </joint>
 	<xacro:soft_hand parent="box" name="soft_hand" left="false" withAdaptiveTransmission="false">
 		<origin xyz="0. 0. 1." rpy="0 0 0"/>

File: soft_hand_description/model/soft_hand.transmission.xacro (robot description, xacro)
@@ -16,5 +16,5 @@
         <type>transmission_interface/SimpleTransmission</type>
         <joint name="${name}_${finger}_inner_joint">
-          <hardwareInterface>hardware_interface/PositionJointInterface</hardwareInterface>
+          <hardwareInterface>hardware_interface/EffortJointInterface</hardwareInterface>
         </joint>
         <actuator name="${name}_${finger}_inner_motor">
@@ -26,5 +26,5 @@
         <type>transmission_interface/SimpleTransmission</type>
         <joint name="${name}_${finger}_inner_joint_mimic">
-          <hardwareInterface>hardware_interface/PositionJointInterface</hardwareInterface>
+          <hardwareInterface>hardware_interface/EffortJointInterface</hardwareInterface>
         </joint>
         <actuator name="${name}_${finger}_inner_motor">
@@ -36,5 +36,5 @@
         <type>transmission_interface/SimpleTransmission</type>
         <joint name="${name}_${finger}_middle_joint">
-          <hardwareInterface>hardware_interface/PositionJointInterface</hardwareInterface>
+          <hardwareInterface>hardware_interface/EffortJointInterface</hardwareInterface>
         </joint>
         <actuator name="${name}_${finger}_middle_motor">
@@ -46,5 +46,5 @@
         <type>transmission_interface/SimpleTransmission</type>
         <joint name="${name}_${finger}_middle_joint_mimic">
-          <hardwareInterface>hardware_interface/PositionJointInterface</hardwareInterface>
+          <hardwareInterface>hardware_interface/EffortJointInterface</hardwareInterface>
         </joint>
         <actuator name="${name}_${finger}_middle_motor">
@@ -56,5 +56,5 @@
         <type>transmission_interface/SimpleTransmission</type>
         <joint name="${name}_${finger}_outer_joint">
-          <hardwareInterface>hardware_interface/PositionJointInterface</hardwareInterface>
+          <hardwareInterface>hardware_interface/EffortJointInterface</hardwareInterface>
         </joint>
         <actuator name="${name}_${finger}_outer_motor">
@@ -66,5 +66,5 @@
         <type>transmission_interface/SimpleTransmission</type>
         <joint name="${name}_${finger}_outer_joint_mimic">
-          <hardwareInterface>hardware_interface/PositionJointInterface</hardwareInterface>
+          <hardwareInterface>hardware_interface/EffortJointInterface</hardwareInterface>
         </joint>
         <actuator name="${name}_${finger}_outer_motor">
@@ -79,5 +79,5 @@
           <type>transmission_interface/SimpleTransmission</type>
           <joint name="${name}_thumb_abd_joint">
-            <hardwareInterface>hardware_interface/PositionJointInterface</hardwareInterface>
+            <hardwareInterface>hardware_interface/EffortJointInterface</hardwareInterface>
           </joint>
           <actuator name="${name}_thumb_abd_motor">
@@ -89,5 +89,5 @@
           <type>transmission_interface/SimpleTransmission</type>
           <joint name="${name}_thumb_inner_joint">
-            <hardwareInterface>hardware_interface/PositionJointInterface</hardwareInterface>
+            <hardwareInterface>hardware_interface/EffortJointInterface</hardwareInterface>
           </joint>
           <actuator name="${name}_thumb_inner_motor">
@@ -99,5 +99,5 @@
           <type>transmission_interface/SimpleTransmission</type>
           <joint name="${name}_thumb_inner_joint_mimic">
-            <hardwareInterface>hardware_interface/PositionJointInterface</hardwareInterface>
+            <hardwareInterface>hardware_interface/EffortJointInterface</hardwareInterface>
           </joint>
           <actuator name="${name}_thumb_inner_motor">
@@ -109,5 +109,5 @@
           <type>transmission_interface/SimpleTransmission</type>
           <joint name="${name}_thumb_outer_joint">
-            <hardwareInterface>hardware_interface/PositionJointInterface</hardwareInterface>
+            <hardwareInterface>hardware_interface/EffortJointInterface</hardwareInterface>
           </joint>
           <actuator name="${name}_thumb_outer_motor">
@@ -119,5 +119,5 @@
           <type>transmission_interface/SimpleTransmission</type>
           <joint name="${name}_thumb_outer_joint_mimic">
-            <hardwareInterface>hardware_interface/PositionJointInterface</hardwareInterface>
+            <hardwareInterface>hardware_interface/EffortJointInterface</hardwareInterface>
           </joint>
           <actuator name="${name}_thumb_outer_motor">

File: soft_hand_description/model/soft_hand.urdf.xacro (robot description, xacro)
@@ -22,5 +22,5 @@
 	<xacro:property name="outer_ub" value="45" />
 	<xacro:property name="velocity" value="100" />
-	<xacro:property name="effort" value="100" />
+	<xacro:property name="effort" value="10" />
 	<xacro:property name="damping" value="0.0" />
 	<xacro:property name="friction" value="0.0" />
@@ -32,4 +32,7 @@
 	<xacro:property name="synergy_damping" value="0.0" />
 	<xacro:property name="synergy_friction" value="0.0" />
+	<xacro:property name="rubber_friction_coefficient" value="1.16" />  <!-- True: 1.16 -->
+	<xacro:property name="rubber_contact_stiffness_coefficient" value="1000000.0" />
+	<xacro:property name="rubber_contact_damping_coefficient" value="1.0" />
 	<!-- SOFT FINGER model -->
 	<!-- 4 fingers are equal (index, middle, ring, little) -->
@@ -150,4 +153,9 @@
 		</link>
 		<gazebo reference="${name}_distal_link">
+			<selfCollide>false</selfCollide>
+			<mu1>${rubber_friction_coefficient}</mu1>
+			<mu2>${rubber_friction_coefficient}</mu2>
+			<kp>${rubber_contact_stiffness_coefficient}</kp>
+			<kd>${rubber_contact_damping_coefficient}</kd>
 			<material>Gazebo/Blue</material>
 		</gazebo>
@@ -280,4 +288,9 @@
 		</link>
 		<gazebo reference="${name}_distal_link">
+			<selfCollide>false</selfCollide>
+			<mu1>${rubber_friction_coefficient}</mu1>
+			<mu2>${rubber_friction_coefficient}</mu2>
+			<kp>${rubber_contact_stiffness_coefficient}</kp>
+			<kd>${rubber_contact_damping_coefficient}</kd>
 			<material>Gazebo/Blue</material>
 		</gazebo>
