Commit message: Color

File: soft_hand_description/model/soft_hand.urdf.xacro (robot description, xacro)
@@ -69,5 +69,5 @@
 		</link>
 		<gazebo reference="${name}_knuckle_link">
-			<material>Gazebo/Blue</material>
+			<material>Gazebo/Gold</material>
 		</gazebo>
 		<!-- PROXIMAL PHALANGE -->
@@ -97,5 +97,5 @@
 		</link>
 		<gazebo reference="${name}_proximal_link">
-			<material>Gazebo/Blue</material>
+			<material>Gazebo/Gold</material>
 		</gazebo>
 		<!-- MIDDLE PHALANGE -->
@@ -125,5 +125,5 @@
 		</link>
 		<gazebo reference="${name}_middle_link">
-			<material>Gazebo/Blue</material>
+			<material>Gazebo/Gold</material>
 		</gazebo>
 		<!-- DISTAL PHALANGE -->
@@ -158,5 +158,5 @@
 			<kp>${rubber_contact_stiffness_coefficient}</kp>
 			<kd>${rubber_contact_damping_coefficient}</kd>
-			<material>Gazebo/Blue</material>
+			<material>Gazebo/Gold</material>
 		</gazebo>
 	</xacro:macro>
@@ -191,5 +191,5 @@
 			</link>
 			<gazebo reference="${name}_knuckle_link">
-				<material>Gazebo/Blue</material>
+				<material>Gazebo/Gold</material>
 			</gazebo>
 			<!-- PROXIMAL PHALANGE -->
@@ -230,5 +230,5 @@
 			</link>
 			<gazebo reference="${name}_knuckle_link">
-				<material>Gazebo/Blue</material>
+				<material>Gazebo/Gold</material>
 			</gazebo>
 			<!-- PROXIMAL PHALANGE -->
@@ -260,5 +260,5 @@
 		</link>
 		<gazebo reference="${name}_proximal_link">
-			<material>Gazebo/Blue</material>
+			<material>Gazebo/Gold</material>
 		</gazebo>
 		<!-- DISTAL PHALANGE -->
@@ -293,5 +293,5 @@
 			<kp>${rubber_contact_stiffness_coefficient}</kp>
 			<kd>${rubber_contact_damping_coefficient}</kd>
-			<material>Gazebo/Blue</material>
+			<material>Gazebo/Gold</material>
 		</gazebo>
 	</xacro:macro>
@@ -360,5 +360,5 @@
 		</link>
 		<gazebo reference="${name}_palm_link">
-			<material>Gazebo/White</material>
+			<material>Gazebo/Gold</material>
 		</gazebo>
 		<!-- THUMB AND FINGERS -->
