Commit message: Centered stl's

File: object_spawn/urdf/object.urdf (robot description, URDF)
Before this commit: robot ycb_object, 2 links, 1 joints
Links:
- link object: geometry collision mesh filename=package://object_spawn/meshes/13_apple_t.stl scale=1 1 1; visual mesh filename=package://object_spawn/meshes/13_apple_t.stl scale=1 1 1
Joints:
- joint world_to_object: origin xyz=0.05 0 1.17 rpy=0 0 0 -> xyz=0 0 0 rpy=0 0 0

File: soft_hand_description/model/soft_hand.urdf.xacro (robot description, xacro)
@@ -18,7 +18,7 @@
 	<xacro:property name="inner_ub" value="60" />
 	<xacro:property name="middle_lb" value="0" />
-	<xacro:property name="middle_ub" value="60" />
+	<xacro:property name="middle_ub" value="75" />
 	<xacro:property name="outer_lb" value="0" />
-	<xacro:property name="outer_ub" value="45" />
+	<xacro:property name="outer_ub" value="60" />
 	<xacro:property name="velocity" value="100" />
 	<xacro:property name="effort" value="10" />

Commit message: Collecting data + fixed finger pub

File: object_spawn/urdf/object.urdf (robot description, URDF)
Before this commit: robot ycb_object, 2 links, 1 joints
Links:
- link object: geometry collision mesh filename=package://object_spawn/meshes/25_mug_t.stl scale=1 1 1; visual mesh filename=package://object_spawn/meshes/25_mug_t.stl scale=1 1 1
